File: CAD/controller/controller.kicad_pcb (KiCad board)
At the start: 2 copper layers, 35.6 x 88.9 mm, 8 parts, among them U1 ESP32-DevKitC

Commit message: updating drawings
Routing:
- net Net-(RotEncoder1-Pin_3): track 46.5 -> 50.6 mm
- net Net-(RotEncoder1-Pin_5): track 65.7 -> 67.3 mm
Changed lines of the file:
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@@
     (pad_to_mask_clearance 0)
     (pcbplotparams
-      (layerselection 0x00010fc_ffffffff)
-      (plot_on_all_layers_selection 0x0000000_00000000)
+      (layerselection 0x0000000_fffffffe)
+      (plot_on_all_layers_selection 0x0000000_80000000)
       (disableapertmacros false)
       (usegerberextensions false)
@@
       (hpglpendiameter 15.000000)
       (dxfpolygonmode true)
-      (dxfimperialunits true)
+      (dxfimperialunits false)
       (dxfusepcbnewfont true)
       (psnegative false)
@@
       (sketchpadsonfab false)
       (subtractmaskfromsilk false)
-      (outputformat 1)
+      (outputformat 3)
       (mirror false)
-      (drillshape 1)
+      (drillshape 2)
       (scaleselection 1)
       (outputdirectory "")
@@
     (fp_line (start 12.45 3.4) (end 12.45 -2.35)
       (stroke (width 0.1) (type solid)) (layer "F.Fab"))
-    (pad "1" thru_hole roundrect (at 0 0) (size 1.7 1.95) (drill 0.95) (layers "*.Cu" "*.Mask") (roundrect_rratio 0.147059)
+    (pad "1" thru_hole roundrect (at 0 0) (size 1.7 1.95) (drill 0.95) (layers "*.Cu" "*.Mask") (roundrect_rratio 0.1470588235)
       (net 1 "GND") (pinfunction "Pin_1") (pintype "passive"))
     (pad "2" thru_hole oval (at 2.5 0) (size 1.7 1.95) (drill 0.95) (layers "*.Cu" "*.Mask")
@@
     (fp_line (start 4.95 3.4) (end 4.95 -2.35)
       (stroke (width 0.1) (type solid)) (layer "F.Fab"))
-    (pad "1" thru_hole roundrect (at 0 0) (size 1.7 2) (drill 1) (layers "*.Cu" "*.Mask") (roundrect_rratio 0.147059)
+    (pad "1" thru_hole roundrect (at 0 0) (size 1.7 2) (drill 1) (layers "*.Cu" "*.Mask") (roundrect_rratio 0.1470588235)
       (net 36 "Net-(MOVE_TO_CONVERSION1-Pin_1)") (pinfunction "Pin_1") (pintype "passive"))
     (pad "2" thru_hole oval (at 2.5 0) (size 1.7 2) (drill 1) (layers "*.Cu" "*.Mask")
@@
     (fp_line (start 4.95 3.4) (end 4.95 -2.35)
       (stroke (width 0.1) (type solid)) (layer "F.Fab"))
-    (pad "1" thru_hole roundrect (at 0 0) (size 1.7 2) (drill 1) (layers "*.Cu" "*.Mask") (roundrect_rratio 0.147059)
+    (pad "1" thru_hole roundrect (at 0 0) (size 1.7 2) (drill 1) (layers "*.Cu" "*.Mask") (roundrect_rratio 0.1470588235)
       (net 2 "+5V") (pinfunction "Pin_1") (pintype "passive"))
     (pad "2" thru_hole oval (at 2.5 0) (size 1.7 2) (drill 1) (layers "*.Cu" "*.Mask")
@@
     (fp_line (start 9.95 3.4) (end 9.95 -2.35)
       (stroke (width 0.1) (type solid)) (layer "F.Fab"))
-    (pad "1" thru_hole roundrect (at 0 0) (size 1.7 1.95) (drill 0.95) (layers "*.Cu" "*.Mask") (roundrect_rratio 0.147059)
+    (pad "1" thru_hole roundrect (at 0 0) (size 1.7 1.95) (drill 0.95) (layers "*.Cu" "*.Mask") (roundrect_rratio 0.1470588235)
       (net 31 "Net-(Display1-Pin_1)") (pinfunction "Pin_1") (pintype "passive"))
     (pad "2" thru_hole oval (at 2.5 0) (size 1.7 1.95) (drill 0.95) (layers "*.Cu" "*.Mask")
@@
     (fp_line (start 4.95 3.4) (end 4.95 -2.35)
       (stroke (width 0.1) (type solid)) (layer "F.Fab"))
-    (pad "1" thru_hole roundrect (at 0 0) (size 1.7 2) (drill 1) (layers "*.Cu" "*.Mask") (roundrect_rratio 0.147059)
+    (pad "1" thru_hole roundrect (at 0 0) (size 1.7 2) (drill 1) (layers "*.Cu" "*.Mask") (roundrect_rratio 0.1470588235)
       (net 35 "Net-(SPEED1-Pin_1)") (pinfunction "Pin_1") (pintype "passive"))
     (pad "2" thru_hole oval (at 2.5 0) (size 1.7 2) (drill 1) (layers "*.Cu" "*.Mask")
@@
     (stroke (width 0.1) (type default)) (fill none) (layer "Edge.Cuts"))
   (segment (start 43.26 111.76) (end 43.18 111.76) (width 0.5) (layer "B.Cu") (net 1))
-  (segment (start 33.02 82.93812) (end 33.02 91.4) (width 0.25) (layer "B.Cu") (net 2))
+  (segment (start 33.02 82.93812) (end 33.02 91.4) (width 0.5) (layer "B.Cu") (net 2))
   (segment (start 33.06 82.97812) (end 33.02 82.93812) (width 0.25) (layer "B.Cu") (net 2))
   (segment (start 33.02 91.4) (end 33.06 91.44) (width 0.25) (layer "B.Cu") (net 2))
-  (segment (start 55.17 104.85) (end 58.42 101.6) (width 0.5) (layer "B.Cu") (net 29))
   (segment (start 59.87 56.44812) (end 58.42 54.99812) (width 0.5) (layer "B.Cu") (net 29))
-  (segment (start 46.43 104.85) (end 55.17 104.85) (width 0.5) (layer "B.Cu") (net 29))
+  (segment (start 48.26 106.68) (end 53.34 106.68) (width 0.5) (layer "B.Cu") (net 29))
+  (segment (start 53.34 106.68) (end 58.42 101.6) (width 0.5) (layer "B.Cu") (net 29))
+  (segment (start 43.18 101.6) (end 48.26 106.68) (width 0.5) (layer "B.Cu") (net 29))
   (segment (start 58.42 101.6) (end 59.87 100.15) (width 0.5) (layer "B.Cu") (net 29))
   (segment (start 59.87 100.15) (end 59.87 56.44812) (width 0.5) (layer "B.Cu") (net 29))
-  (segment (start 43.18 101.6) (end 46.43 104.85) (width 0.5) (layer "B.Cu") (net 29))
   (segment (start 50.8 65.15812) (end 58.42 57.53812) (width 0.5) (layer "B.Cu") (net 30))
   (segment (start 49.375 100.175) (end 50.8 101.6) (width 0.5) (layer "B.Cu") (net 30))
@@
   (segment (start 48.26 111.76) (end 53.34 111.76) (width 0.5) (layer "B.Cu") (net 33))
   (segment (start 53.34 111.76) (end 61.184486 103.915514) (width 0.5) (layer "B.Cu") (net 33))
-  (segment (start 38.18 101.6) (end 47.721522 92.058478) (width 0.5) (layer "B.Cu") (net 34))
+  (segment (start 38.18 101.6) (end 38.18 98.98) (width 0.5) (layer "B.Cu") (net 34))
+  (segment (start 38.18 98.98) (end 40.64 96.52) (width 0.5) (layer "B.Cu") (net 34))
   (segment (start 47.721522 79.859642) (end 33.02 65.15812) (width 0.5) (layer "B.Cu") (net 34))
-  (segment (start 47.721522 92.058478) (end 47.721522 79.859642) (width 0.5) (layer "B.Cu") (net 34))
+  (segment (start 47.721522 96.52) (end 47.721522 79.859642) (width 0.5) (layer "B.Cu") (net 34))
+  (segment (start 40.64 96.52) (end 47.721522 96.52) (width 0.5) (layer "B.Cu") (net 34))
   (segment (start 43.22 77.89812) (end 33.02 67.69812) (width 0.5) (layer "B.Cu") (net 35))
   (segment (start 43.22 91.44) (end 43.22 77.89812) (width 0.5) (layer "B.Cu") (net 35))
@@
   (segment (start 53.38 91.44) (end 53.38 70.19812) (width 0.5) (layer "B.Cu") (net 36))
   (zone (net 1) (net_name "GND") (layer "B.Cu") (hatch edge 0.5)
-    (connect_pads (clearance 0.5))
+    (connect_pads yes (clearance 0.5))
     (min_thickness 0.25) (filled_areas_thickness no)
     (fill yes (thermal_gap 0.5) (thermal_bridge_width 0.5))
     (polygon
       (pts
+        (xy 63.5 27.94)
         (xy 63.5 116.84)
         (xy 27.94 116.84)
         (xy 27.94 27.94)
-        (xy 63.5 27.94)
       )
     )

Commit message: Updated PCB
Parts:
- moved Display1 76.2 mm to (43.3, 35.6)
- moved RotEncoder1 55.9 mm to (33.0, 45.7)
- moved C1 55.3 mm to (58.4, 46.3), turned to 90 degrees
- moved C2 55.3 mm to (50.8, 46.3), turned to 90 degrees
- moved MOVE_TO_CONVERSION1 35.6 mm to (53.3, 55.9)
- moved POWER1 35.6 mm to (33.0, 55.9)
- moved SPEED1 35.6 mm to (43.2, 55.9)
- moved U1 31.4 mm to (33.0, 68.6)
Routing:
- net GND: track 0.08 -> 97.9 mm
- net +5V: track 8.58 -> 59.9 mm
- net Net-(RotEncoder1-Pin_5): track 67.3 -> 16.9 mm
- net Net-(RotEncoder1-Pin_4): track 58.5 -> 15.7 mm
- net Net-(Display1-Pin_1): track 79.9 -> 40.2 mm
- net Net-(Display1-Pin_3): track 86.1 -> 46.7 mm
- net Net-(SPEED1-Pin_1): track 28.0 -> 47.4 mm
- net Net-(Display1-Pin_4): track 71.3 -> 53.5 mm
- net Net-(MOVE_TO_CONVERSION1-Pin_1): track 28.4 -> 42.7 mm
- net Net-(RotEncoder1-Pin_3): track 50.6 -> 53.0 mm
- removed copper zone on B.Cu, net GND
